Commit message: fixing errors

File: my_robot/urdf/my_robot.xacro (robot description, xacro)
@@ -177,3 +177,12 @@
     </visual>
   </link>
+  <gazebo reference="left_wheel">
+    <material>Gazebo/Black</material>
+  </gazebo>
+  <gazebo reference="chassis">
+    <material>Gazebo/Red</material>
+  </gazebo>
+  <gazebo reference="right_wheel">
+    <material>Gazebo/Green</material>
+  </gazebo>
 </robot>
